Commit message: base_link corrupt

File: src/my_simrobot/urdf/robot.urdf.xacro (robot description, xacro)
@@ -8,4 +8,6 @@
   <xacro:include filename="$(find my_simrobot)/urdf/simrobot_description.gazebo"/>
   <xacro:include filename="$(find my_simrobot)/urdf/rplidar_laser.gazebo.xacro" />
+  <xacro:include filename="$(find aubo_description)/urdf/aubo_i5_robot_gazebo.urdf.xacro" />
+  <!-- <xacro:include filename="$(find aubo_description)/urdf/aubo_i5.urdf.xacro" /> -->
   <!--<xacro:hokuyo_lx30_laser_gazebo_v0 name="${name}" ros_topic="${ros_topic}" update_rate="${update_rate}" min_angle="${min_angle}" max_angle="${max_angle}" />-->
 </robot>

File: src/my_simrobot/urdf/simrobot_description.urdf (robot description, URDF)
Before this commit: robot simrobot, 5 links, 4 joints
Links:
- removed link base_link
- added link mobile_link, mass 0.62461; collision mesh filename=package://my_simrobot/meshes/base_link.STL; visual mesh filename=package://my_simrobot/meshes/base_link.STL

Commit message: try to use group in launch to combine grip with robot

File: src/my_simrobot/urdf/robot.urdf.xacro (robot description, xacro)
@@ -8,5 +8,5 @@
   <xacro:include filename="$(find my_simrobot)/urdf/simrobot_description.gazebo"/>
   <xacro:include filename="$(find my_simrobot)/urdf/rplidar_laser.gazebo.xacro" />
-  <xacro:include filename="$(find aubo_description)/urdf/aubo_i5_robot_gazebo.urdf.xacro" />
+  <!-- <xacro:include filename="$(find aubo_description)/urdf/aubo_i5_robot_gazebo.urdf.xacro" /> -->
   <!-- <xacro:include filename="$(find aubo_description)/urdf/aubo_i5.urdf.xacro" /> -->
   <!--<xacro:hokuyo_lx30_laser_gazebo_v0 name="${name}" ros_topic="${ros_topic}" update_rate="${update_rate}" min_angle="${min_angle}" max_angle="${max_angle}" />-->

File: src/my_simrobot/urdf/simrobot_description.urdf (robot description, URDF)
Before this commit: robot simrobot, 5 links, 4 joints
Links:
- removed link mobile_link
- added link base_link, mass 0.62461; collision mesh filename=package://my_simrobot/meshes/base_link.STL; visual mesh filename=package://my_simrobot/meshes/base_link.STL
