Commit message: try to solve moveit config

File: src/car4wd/urdf/car4wd.urdf (robot description, URDF)
Before this commit: robot car4wd, 16 links, 15 joints
Links:
- added link left_sonar; collision box size=0.01 0.04 0.04; collision cylinder length=0.01 radius=0.01
- added link usb_camera_link, mass 0.1; collision box size=0.01 0.04 0.04; visual box size=0.01 0.04 0.04
Joints:
- added joint base_to_camera_joint: type fixed, parent base_link, child usb_camera_link, origin xyz=0.1 0.2 0.22 rpy=0 0 0
- added joint left_sonar_joint: type fixed, parent base_link, child left_sonar, origin xyz=0.28 0 0.16 rpy=0 0 0
