Commit message: start new version of car4wd

File: src/mobile_manipulator/car4wd/urdf/car4wd.xacro (robot description, xacro)
@@ -5,7 +5,14 @@
   xmlns:xacro="http://ros.org/wiki/xacro"
   name="robot_urdf.gazebo">
-  <xacro:include filename="$(find car4wd)/urdf/car4wd.urdf"/>
+  <xacro:include filename="$(find car4wd)/urdf/car4wd.urdf.xacro"/>
   <xacro:include filename="$(find car4wd)/urdf/car4wd.gazebo"/>
-  <xacro:include filename="$(find car4wd)/urdf/rplidar_laser.gazebo.xacro" />
-  <!--<xacro:hokuyo_lx30_laser_gazebo_v0 name="${name}" ros_topic="${ros_topic}" update_rate="${update_rate}" min_angle="${min_angle}" max_angle="${max_angle}" />-->
+  <xacro:include filename="$(find car4wd)/urdf/aubo_i5.urdf.xacro"/>
+  <!--xacro:include filename="$(find car4wd)/urdf/rplidar_laser.gazebo.xacro"/-->
+<xacro:aubo_i5_robot prefix=""/>
+<xacro:car />
+  <joint name="world_joint" type="fixed">
+    <parent link="base_link"/>
+    <child link="base_Link"/>
+    <origin xyz="0.0 0.0 0.2" rpy="0.0 0.0 0.0" />
+  </joint>
 </robot>

Commit message: add controller but move_base is still in

File: src/mobile_manipulator/car4wd/urdf/car4wd.xacro (robot description, xacro)
@@ -5,14 +5,7 @@
   xmlns:xacro="http://ros.org/wiki/xacro"
   name="robot_urdf.gazebo">
-  <xacro:include filename="$(find car4wd)/urdf/car4wd.urdf.xacro"/>
+  <xacro:include filename="$(find car4wd)/urdf/car4wd.urdf"/>
   <xacro:include filename="$(find car4wd)/urdf/car4wd.gazebo"/>
-  <xacro:include filename="$(find car4wd)/urdf/aubo_i5.urdf.xacro"/>
-  <!--xacro:include filename="$(find car4wd)/urdf/rplidar_laser.gazebo.xacro"/-->
-<xacro:aubo_i5_robot prefix=""/>
-<xacro:car />
-  <joint name="world_joint" type="fixed">
-    <parent link="base_link"/>
-    <child link="base_Link"/>
-    <origin xyz="0.0 0.0 0.2" rpy="0.0 0.0 0.0" />
-  </joint>
+  <xacro:include filename="$(find car4wd)/urdf/rplidar_laser.gazebo.xacro" />
+  <!--<xacro:hokuyo_lx30_laser_gazebo_v0 name="${name}" ros_topic="${ros_topic}" update_rate="${update_rate}" min_angle="${min_angle}" max_angle="${max_angle}" />-->
 </robot>
